Commit message: feat(usb): 打通 USB 动态状态与底盘控制链路
- STM32 新增 0x83 WheelState / 0x84 ImuState，4 相 5 ms 调度，
  每 tick 只发一帧避免 CDC TX 丢帧
- 底盘消费 UnifiedCmd：CMD_VALID|CMD_MOTION_ENABLE + 100 ms 新鲜度门控，
  超时/非法立即 force_stop，并锁存 usb_armed
- AppChassisDiag 增加四轮位置/力矩/温度/状态，修复 chassis target 误置
  gimbal/INS 状态位
- ROS 新增 ChassisState.msg，usb_bridge 发布 /chassis/state、/imu/data、
  serial/joint_states_raw、/diagnostics，保留 /usb_bridge/state
- 新增 cmd_vel_to_unified，默认 enable_motion=false；sentry.launch 新增
  chassis_transport:=usb|udp
- 麦轮 URDF 四轮改 continuous，新增 imu_link
- 实测：四轮 0.05 m/s 跟随、/joint_states 正确、零速/超时/门控通过

Co-Authored-By: Claude Code <noreply@anthropic.com>

File: ros_ws/src/sentry_description/urdf/mecanum_static.urdf (robot description, URDF)
Before this commit: robot sentry_mecanum, 8 links, 7 joints
Links:
- added link imu_link
Joints:
- added joint imu_link_joint: type fixed, parent base_link, child imu_link, origin xyz=0 0 0 rpy=0 0 0
- joint wheel_back_left_joint: axis (none) -> 0 1 0; limit (none) -> effort=10.0 velocity=45.0; type fixed -> continuous
- joint wheel_back_right_joint: axis (none) -> 0 1 0; limit (none) -> effort=10.0 velocity=45.0; type fixed -> continuous
- joint wheel_front_left_joint: axis (none) -> 0 1 0; limit (none) -> effort=10.0 velocity=45.0; type fixed -> continuous
- joint wheel_front_right_joint: axis (none) -> 0 1 0; limit (none) -> effort=10.0 velocity=45.0; type fixed -> continuous

Commit message: fix(perception): 修正 MID360 yaw 并标定代价地图
- URDF: front_mid360 yaw -90° → 0°（实测物理前方被映射到右扇区）
- 代价地图: terrain intensity 实际是高度差，过滤范围改为 0.0–5.0；
  observation_persistence 1.5 s，terrain decayTime 1.0 s；
  箱子标定 60 cm，地形误差约 1 cm，代价地图误差约 1 格
- RViz: 仅调整颜色（全局路径红、局部路径蓝、扫描绿）；
  新增 rviz_config 参数和灰度代价地图备选配置
- 文档: 接手文档同步 MID360 yaw、配色与标定结果

Co-Authored-By: Claude Code <noreply@anthropic.com>

File: ros_ws/src/sentry_description/urdf/mecanum_static.urdf (robot description, URDF)
Before this commit: robot sentry_mecanum, 9 links, 8 joints
Joints:
- joint front_mid360_joint: origin xyz=0.15 0 0.165 rpy=0 0 -1.57079632679 -> xyz=0.15 0 0.165 rpy=0 0 0
